File: v_0.1/hardware/good-peater/good-peater.kicad_sch (KiCad schematic)
At the start: 52 parts, among them Q1 SSM3J332R, Q2 FDS6675BZ, Q3 SSM3J332R, Q4 SSM3J332R, Q5 MMUN2211LT1G, U1 CN3801, U1 LM2903, U3 TCM810

Commit message: update
Parts:
- added C11: 0.1uF 50V, Capacitor_SMD:C_0805_2012Metric, symbol Device:C
- added J1: Conn_01x02_Socket, Connector_JST:JST_PH_B2B-PH-K_1x02_P2.00mm_Vertical, symbol Connector:Conn_01x02_Socket
Connections:
- net GND: now also BNEG1.1 (BAT_NEG), C10.2, C12.2, HEAT.1 (K), R2.1, R4.1, THRM.2, U1.4 (V-), U3.1 (GND), C11.2, J1.2 (Pin_2)
- net SOLAR+: now also Q1.2 (S), R1.1, R14.1, R3.1, R6.2, R7.2, U1.8 (V+), C11.1
- net at HEAT.2 (A): now also R19.2
- net at Q3.1 (G): now also U3.2 (RESET)
- net BAT: now reaches Q3.2 (S)
- net BAT: now also BPOS1.1 (BAT_POS), C13.1, Q4.2 (S), R18.1, U3.3 (V_{DD}), J1.1 (Pin_1)
- net at Q3.3 (D): now also F2.1
- net LOAD+: now reaches C10.1
- net LOAD+: now also F2.2
- net at R3.2: now also R4.2, R5.2, U1.3 (+)
- net at U1.5 (+): now also R1.2, R13.1, R2.2, THRM.1, U1.2 (-)
- net at U1.6 (-): now also R7.1
- net at U1.7: now also D1.1, R13.2, R14.2
- net at U1.1: now also D1.2, Q1.1 (G), R5.1, R6.1
- net at F1.1: now also Q1.3 (D), R19.1
- net HEATER+: now reaches F1.2
- net HEATER+: now also C12.1
Other:
- note added: "~OVERTEMP~"
- note added: "~UNDERTEMP~"
- moved on the sheet: BNEG1, BPOS1, C1, C10, C12, C13, C2, C3, C4, C6, C7, C8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
